File: A/Hardware/PC104/MAG_Plus/FEMTO.sch (KiCad schematic (older format))
At the start: 10 parts, among them J6 Conn_01x12_Male, U11 ISO7341C

Commit message: PCB update
Connections:
- net FOD_VAUX is gone; now on net FOD_3V3: J6.7 (Pin_7)
Changed lines of the file:
@@
 GND
 Text GLabel 10300 2450 0    50   Input ~ 0
-FOD_VAUX
+FOD_3V3
 Text GLabel 10300 2350 0    50   Input ~ 0
 FOD_DPL

Commit message: Update PCBs
New version of PCBs
Parts:
- added JP33: Jumper_2_Open, Jumper:SolderJumper-2_P1.3mm_Open_RoundedPad1.0x1.5mm, symbol Jumper:Jumper_2_Open
Connections:
- net FOD_SDA: now also JP33.2 (B)
- new net FOD_STS: JP33.1 (A)
Changed lines of the file:
@@
 Text Notes 10600 7650 0    79   ~ 0
 A
+$Comp
+L Jumper:Jumper_2_Open JP33
+U 1 1 6179DF88
+P 8800 4250
+F 0 "JP33" H 8800 4485 50  0000 C CNN
+F 1 "Jumper_2_Open" H 8800 4394 50  0000 C CNN
+F 2 "Jumper:SolderJumper-2_P1.3mm_Open_RoundedPad1.0x1.5mm" H 8800 4250 50  0001 C CNN
+F 3 "~" H 8800 4250 50  0001 C CNN
+	1    8800 4250
+	1    0    0    -1
+$EndComp
+Text GLabel 9000 4250 2    50   Input ~ 0
+FOD_SDA
+Text GLabel 8600 4250 0    50   Input ~ 0
+FOD_STS
 $EndSCHEMATC
