File: A/Hardware/PC104/MAG_Plus/MAG_Plus.kicad_pcb (KiCad board)
At the start: 2 copper layers, 96 x 89.9 mm, 106 parts, among them J1 RPi_GPIO, J2 U.FL-R-SMT(01), J3 U.FL-R-SMT(01), J4 U.FL-R-SMT(01), J5 U.FL-R-SMT(01), J6 Conn_01x12_Male, J7 Conn_01x04_Male, J8 Conn_01x04_Male, J9 Conn_01x06_Male, SW1 SW_Push, U1 Payload, U10 QPQ1906SR, U11 ISO7341C, U12 PIC16F1847-I_SO, U13 LP38693MP-3.3, U14 LP38693MP-3.3, U15 LP38693MP-5.0, U16 LP38693MP-3.3, U2 ISO1540, U3 ISO7341C, U4 AD8302, U5 AD8302, U6 AD7904BRUZ-REEL7, U7 QPQ1906SR, U8 QPQ1906SR, U9 QPQ1906SR

Commit message: Update PCB A
Parts:
- moved C5 6.77 mm to (123.0, 74.0), turned to 180 degrees
- moved C6 6.76 mm to (129.5, 74.0)
Routing:
- net PIC_SCL: track 76.1 -> 68.3 mm
- net PIC_3V3: track 146.0 -> 142.7 mm
- net CSP_SCL: track 13.7 -> 15.7 mm
- net SAT_3V3: track 31.9 -> 33.2 mm
- net FOD_SCK: track 31.2 -> 31.8 mm
- net FOD_MOSI: track 31.3 -> 31.9 mm
- net GND: vias 15 -> 16

Commit message: new modifications pcb
Parts:
- moved SW1 5.43 mm to (193.2, 94.6)
Routing:
- net MCLR: track 116.4 -> 109.5 mm
- net MAG_3V3: track 113.9 -> 113.3 mm
- net RPI_SDA: track 122.3 -> 121.8 mm
- net RPI_SCL: track 120.8 -> 120.3 mm
Other:
- board size 96 x 89.9 mm -> 92.5 x 86.8 mm

Commit message: More PCB Changes
Connections:
- C6 pad 1: PIC_3V3 -> PIC_3V3J
- R5 pad 1: PIC_3V3 -> PIC_3V3J
- R6 pad 1: PIC_3V3 -> PIC_3V3J
- U2 pad 8: PIC_3V3 -> PIC_3V3J
Routing:
- net AOA_5V: track 73.8 -> 136.0 mm, vias 2 -> 4
- net PIC_3V3: track 142.7 -> 105.5 mm
- net PIC_3V3J: track 19.8 -> 35.8 mm
- net MAG_3V3: track 113.3 -> 115.0 mm, vias 1 -> 2
- net PIC_EN: track 34.4 -> 33.8 mm
- net VMAG2: track 47.4 -> 46.8 mm
- net AOA_EN: track 42.9 -> 43.4 mm
- net VIN: track 283.2 -> 283.7 mm

Commit message: PCB update
Parts:
- removed C28, C29, C30: C, Capacitors_SMD:C_0402
- removed R12, R14: R, Resistors_SMD:R_0402
- removed U6: AD7904BRUZ-REEL7, Housings_SSOP:TSSOP-16_4.4x5mm_Pitch0.65mm
- added G***: LOGO, L86:SPEL_logo, B.Cu at (104.3, 83.4)
- added J10: Conn_01x04_Male, Connectors_Molex:Molex_PicoBlade_53398-0471_04x1.25mm_Straight, F.Cu at (192.2, 265.6)
- added J10: Conn_01x04_Male, Connectors_Molex:Molex_PicoBlade_53398-0471_04x1.25mm_Straight, F.Cu at (268.7, 55.2)
- added J11: Conn_01x04_Male, Connectors_Molex:Molex_PicoBlade_53398-0471_04x1.25mm_Straight, F.Cu at (475.7, 56.0)
- added J11: Conn_01x04_Male, Connectors_Molex:Molex_PicoBlade_53398-0471_04x1.25mm_Straight, F.Cu at (192.1, 158.2)
- added J12: Conn_01x07_Female, Pin_Headers:Pin_Header_Straight_1x07_Pitch2.54mm_SMD_Pin1Left, F.Cu at (174.4, 297.1)
- added J12: Conn_01x07_Female, Pin_Headers:Pin_Header_Straight_1x07_Pitch2.54mm_SMD_Pin1Left, F.Cu at (300.6, 65.8)
- added J13: Conn_01x07_Female, Pin_Headers:Pin_Header_Straight_1x07_Pitch2.54mm_SMD_Pin1Right, F.Cu at (496.8, 63.4)
- added J13: Conn_01x07_Female, Pin_Headers:Pin_Header_Straight_1x07_Pitch2.54mm_SMD_Pin1Right, F.Cu at (174.4, 179.9)
- added J14: Conn_01x07_Female, Pin_Headers:Pin_Header_Straight_1x07_Pitch2.54mm_SMD_Pin1Left, F.Cu at (151.4, 297.1)
- added J14: Conn_01x07_Female, Pin_Headers:Pin_Header_Straight_1x07_Pitch2.54mm_SMD_Pin1Left, F.Cu at (300.5, 88.8)
- added J15: Conn_01x07_Female, Pin_Headers:Pin_Header_Straight_1x07_Pitch2.54mm_SMD_Pin1Right, F.Cu at (496.8, 86.4)
- added J15: Conn_01x07_Female, Pin_Headers:Pin_Header_Straight_1x07_Pitch2.54mm_SMD_Pin1Right, F.Cu at (151.4, 179.9)
- added JP19: Jumper_3_Open, Jumper:SolderJumper-3_P1.3mm_Open_RoundedPad1.0x1.5mm, F.Cu at (146.6, 303.4)
- added JP19: Jumper_3_Open, Jumper:SolderJumper-3_P1.3mm_Open_RoundedPad1.0x1.5mm, F.Cu at (306.9, 93.6)
- added JP20: Jumper_3_Open, Jumper:SolderJumper-3_P1.3mm_Open_RoundedPad1.0x1.5mm, F.Cu at (503.1, 91.3)
- added JP20: Jumper_3_Open, Jumper:SolderJumper-3_P1.3mm_Open_RoundedPad1.0x1.5mm, F.Cu at (146.5, 186.2)
- added JP21: Jumper_3_Open, Jumper:SolderJumper-3_P1.3mm_Open_RoundedPad1.0x1.5mm, F.Cu at (143.7, 303.4)
- added JP21: Jumper_3_Open, Jumper:SolderJumper-3_P1.3mm_Open_RoundedPad1.0x1.5mm, F.Cu at (306.8, 96.5)
- added JP22: Jumper_3_Open, Jumper:SolderJumper-3_P1.3mm_Open_RoundedPad1.0x1.5mm, F.Cu at (503.1, 94.2)
- added JP22: Jumper_3_Open, Jumper:SolderJumper-3_P1.3mm_Open_RoundedPad1.0x1.5mm, F.Cu at (143.6, 186.2)
- added JP23: Jumper_3_Open, Jumper:SolderJumper-3_P1.3mm_Open_RoundedPad1.0x1.5mm, F.Cu at (497.6, 91.2)
- added JP23: Jumper_3_Open, Jumper:SolderJumper-3_P1.3mm_Open_RoundedPad1.0x1.5mm, F.Cu at (146.6, 178.7)
- added JP24: Jumper_3_Open, Jumper:SolderJumper-3_P1.3mm_Open_RoundedPad1.0x1.5mm, F.Cu at (497.6, 96.9)
- added JP24: Jumper_3_Open, Jumper:SolderJumper-3_P1.3mm_Open_RoundedPad1.0x1.5mm, F.Cu at (140.8, 178.7)
- added JP25: Jumper_3_Open, Jumper:SolderJumper-3_P1.3mm_Open_RoundedPad1.0x1.5mm, F.Cu at (146.6, 295.9)
- added JP25: Jumper_3_Open, Jumper:SolderJumper-3_P1.3mm_Open_RoundedPad1.0x1.5mm, F.Cu at (299.3, 93.6)
- added JP26: Jumper_3_Open, Jumper:SolderJumper-3_P1.3mm_Open_RoundedPad1.0x1.5mm, F.Cu at (140.9, 295.9)
- added JP26: Jumper_3_Open, Jumper:SolderJumper-3_P1.3mm_Open_RoundedPad1.0x1.5mm, F.Cu at (299.3, 99.3)
- added JP27: Jumper_3_Open, Jumper:SolderJumper-3_P1.3mm_Open_RoundedPad1.0x1.5mm, F.Cu at (497.6, 94.1)
- added JP27: Jumper_3_Open, Jumper:SolderJumper-3_P1.3mm_Open_RoundedPad1.0x1.5mm, F.Cu at (143.7, 178.7)
- added JP28: Jumper_3_Open, Jumper:SolderJumper-3_P1.3mm_Open_RoundedPad1.0x1.5mm, F.Cu at (143.8, 295.8)
- added JP28: Jumper_3_Open, Jumper:SolderJumper-3_P1.3mm_Open_RoundedPad1.0x1.5mm, F.Cu at (299.2, 96.5)
- added R16: R, Resistors_SMD:R_0402, F.Cu at (504.4, 59.0)
- added R16: R, Resistors_SMD:R_0402, F.Cu at (178.8, 187.5)
- added R17: R, Resistors_SMD:R_0402, F.Cu at (178.8, 304.8)
- added R17: R, Resistors_SMD:R_0402, F.Cu at (308.2, 61.4)
- added R18: R, Resistors_SMD:R_0402, F.Cu at (499.3, 59.0)
- added R18: R, Resistors_SMD:R_0402, F.Cu at (178.8, 182.4)
- added R19: R, Resistors_SMD:R_0402, F.Cu at (178.8, 299.7)
- added R19: R, Resistors_SMD:R_0402, F.Cu at (303.1, 61.4)
- added REF**: MountingHole_2.7mm_M2.5_ISO14580_Pad, Mounting_Holes:MountingHole_2.7mm_M2.5_ISO14580_Pad, F.Cu at (553.3, 45.9)
- added REF**: MountingHole_2.7mm_M2.5_ISO14580_Pad, Mounting_Holes:MountingHole_2.7mm_M2.5_ISO14580_Pad, F.Cu at (346.6, 109.4)
- added REF**: MountingHole_2.7mm_M2.5_ISO14580_Pad, Mounting_Holes:MountingHole_2.7mm_M2.5_ISO14580_Pad, F.Cu at (242.8, 109.4)
- added REF**: MountingHole_2.7mm_M2.5_ISO14580_Pad, Mounting_Holes:MountingHole_2.7mm_M2.5_ISO14580_Pad, F.Cu at (242.8, 45.2)
- added REF**: MountingHole_2.7mm_M2.5_ISO14580_Pad, Mounting_Holes:MountingHole_2.7mm_M2.5_ISO14580_Pad, F.Cu at (151.3, 45.2)
- added REF**: MountingHole_2.7mm_M2.5_ISO14580_Pad, Mounting_Holes:MountingHole_2.7mm_M2.5_ISO14580_Pad, F.Cu at (150.9, 109.4)
- added REF**: MountingHole_2.2mm_M2_DIN965_Pad, Mounting_Holes:MountingHole_2.2mm_M2_DIN965_Pad, F.Cu at (336.1, 46.0)
- added REF**: MountingHole_2.2mm_M2_DIN965_Pad, Mounting_Holes:MountingHole_2.2mm_M2_DIN965_Pad, F.Cu at (293.5, 108.6)
- added REF**: MountingHole_2.2mm_M2_DIN965_Pad, Mounting_Holes:MountingHole_2.2mm_M2_DIN965_Pad, F.Cu at (293.5, 46.0)
- added REF**: MountingHole_2.2mm_M2_DIN965_Pad, Mounting_Holes:MountingHole_2.2mm_M2_DIN965_Pad, F.Cu at (336.1, 108.6)
- added REF**: MountingHole_2.2mm_M2_DIN965_Pad, Mounting_Holes:MountingHole_2.2mm_M2_DIN965_Pad, F.Cu at (194.2, 332.7)
- added REF**: MountingHole_2.7mm_M2.5_ISO14580_Pad, Mounting_Holes:MountingHole_2.7mm_M2.5_ISO14580_Pad, F.Cu at (461.8, 45.9)
- added REF**: MountingHole_2.2mm_M2_DIN965_Pad, Mounting_Holes:MountingHole_2.2mm_M2_DIN965_Pad, F.Cu at (131.6, 332.7)
- added REF**: MountingHole_2.2mm_M2_DIN965_Pad, Mounting_Holes:MountingHole_2.2mm_M2_DIN965_Pad, F.Cu at (194.2, 290.1)
- added REF**: MountingHole_2.2mm_M2_DIN965_Pad, Mounting_Holes:MountingHole_2.2mm_M2_DIN965_Pad, F.Cu at (131.6, 290.1)
- added REF**: MountingHole_2.7mm_M2.5_ISO14580_Pad, Mounting_Holes:MountingHole_2.7mm_M2.5_ISO14580_Pad, F.Cu at (547.0, 53.4)
- added REF**: MountingHole_2.7mm_M2.5_ISO14580_Pad, Mounting_Holes:MountingHole_2.7mm_M2.5_ISO14580_Pad, F.Cu at (547.0, 101.3)
- added REF**: MountingHole_2.7mm_M2.5_ISO14580_Pad, Mounting_Holes:MountingHole_2.7mm_M2.5_ISO14580_Pad, F.Cu at (512.0, 42.8)
- added REF**: MountingHole_2.7mm_M2.5_ISO14580_Pad, Mounting_Holes:MountingHole_2.7mm_M2.5_ISO14580_Pad, F.Cu at (512.0, 113.1)
- added REF**: MountingHole_5.3mm_M5_DIN965_Pad, Mounting_Holes:MountingHole_5.3mm_M5_DIN965_Pad, F.Cu at (314.8, 107.8)
- added REF**: MountingHole_5.3mm_M5_DIN965_Pad, Mounting_Holes:MountingHole_5.3mm_M5_DIN965_Pad, F.Cu at (314.8, 46.8)
- added REF**: MountingHole_5.3mm_M5_DIN965_Pad, Mounting_Holes:MountingHole_5.3mm_M5_DIN965_Pad, F.Cu at (132.4, 311.4)
- added REF**: MountingHole_2.7mm_M2.5_ISO14580_Pad, Mounting_Holes:MountingHole_2.7mm_M2.5_ISO14580_Pad, F.Cu at (553.3, 110.1)
- added REF**: MountingHole_5.3mm_M5_DIN965_Pad, Mounting_Holes:MountingHole_5.3mm_M5_DIN965_Pad, F.Cu at (193.4, 311.4)
- added REF**: MountingHole_2.7mm_M2.5_ISO14580_Pad, Mounting_Holes:MountingHole_2.7mm_M2.5_ISO14580_Pad, F.Cu at (201.0, 251.7)
- added REF**: MountingHole_2.7mm_M2.5_ISO14580_Pad, Mounting_Holes:MountingHole_2.7mm_M2.5_ISO14580_Pad, F.Cu at (201.0, 343.3)
- added REF**: MountingHole_2.7mm_M2.5_ISO14580_Pad, Mounting_Holes:MountingHole_2.7mm_M2.5_ISO14580_Pad, F.Cu at (124.8, 251.7)
- added REF**: MountingHole_2.7mm_M2.5_ISO14580_Pad, Mounting_Holes:MountingHole_2.7mm_M2.5_ISO14580_Pad, F.Cu at (124.8, 343.3)
- added REF**: MountingHole_2.7mm_M2.5_ISO14580_Pad, Mounting_Holes:MountingHole_2.7mm_M2.5_ISO14580_Pad, F.Cu at (115.3, 251.4)
- added REF**: MountingHole_2.7mm_M2.5_ISO14580_Pad, Mounting_Holes:MountingHole_2.7mm_M2.5_ISO14580_Pad, F.Cu at (115.3, 343.0)
- added REF**: MountingHole_2.7mm_M2.5_ISO14580_Pad, Mounting_Holes:MountingHole_2.7mm_M2.5_ISO14580_Pad, F.Cu at (39.1, 251.4)
- added REF**: MountingHole_2.7mm_M2.5_ISO14580_Pad, Mounting_Holes:MountingHole_2.7mm_M2.5_ISO14580_Pad, F.Cu at (39.1, 343.0)
- added REF**: MountingHole_2.7mm_M2.5_ISO14580_Pad, Mounting_Holes:MountingHole_2.7mm_M2.5_ISO14580_Pad, F.Cu at (115.4, 144.2)
- added REF**: MountingHole_2.7mm_M2.5_ISO14580_Pad, Mounting_Holes:MountingHole_2.7mm_M2.5_ISO14580_Pad, F.Cu at (452.1, 45.9)
- added REF**: MountingHole_2.7mm_M2.5_ISO14580_Pad, Mounting_Holes:MountingHole_2.7mm_M2.5_ISO14580_Pad, F.Cu at (115.4, 235.8)
- added REF**: MountingHole_2.7mm_M2.5_ISO14580_Pad, Mounting_Holes:MountingHole_2.7mm_M2.5_ISO14580_Pad, F.Cu at (39.2, 144.2)
- added REF**: MountingHole_2.7mm_M2.5_ISO14580_Pad, Mounting_Holes:MountingHole_2.7mm_M2.5_ISO14580_Pad, F.Cu at (39.2, 235.8)
- added REF**: MountingHole_2.7mm_M2.5_ISO14580_Pad, Mounting_Holes:MountingHole_2.7mm_M2.5_ISO14580_Pad, F.Cu at (187.4, 230.1)
- added REF**: MountingHole_2.7mm_M2.5_ISO14580_Pad, Mounting_Holes:MountingHole_2.7mm_M2.5_ISO14580_Pad, F.Cu at (139.6, 230.1)
- added REF**: MountingHole_2.7mm_M2.5_ISO14580_Pad, Mounting_Holes:MountingHole_2.7mm_M2.5_ISO14580_Pad, F.Cu at (198.1, 195.1)
- added REF**: MountingHole_2.7mm_M2.5_ISO14580_Pad, Mounting_Holes:MountingHole_2.7mm_M2.5_ISO14580_Pad, F.Cu at (127.8, 195.1)
- added REF**: MountingHole_2.7mm_M2.5_ISO14580_Pad, Mounting_Holes:MountingHole_2.7mm_M2.5_ISO14580_Pad, F.Cu at (201.0, 235.8)
- added REF**: MountingHole_2.7mm_M2.5_ISO14580_Pad, Mounting_Holes:MountingHole_2.7mm_M2.5_ISO14580_Pad, F.Cu at (124.8, 235.8)
- added REF**: MountingHole_2.7mm_M2.5_ISO14580_Pad, Mounting_Holes:MountingHole_2.7mm_M2.5_ISO14580_Pad, F.Cu at (201.0, 144.2)
- added REF**: MountingHole_2.7mm_M2.5_ISO14580_Pad, Mounting_Holes:MountingHole_2.7mm_M2.5_ISO14580_Pad, F.Cu at (360.6, 45.9)
- added REF**: MountingHole_2.7mm_M2.5_ISO14580_Pad, Mounting_Holes:MountingHole_2.7mm_M2.5_ISO14580_Pad, F.Cu at (124.8, 144.2)
- added REF**: MountingHole_2.7mm_M2.5_ISO14580_Pad, Mounting_Holes:MountingHole_2.7mm_M2.5_ISO14580_Pad, F.Cu at (360.6, 110.1)
- added REF**: MountingHole_2.7mm_M2.5_ISO14580_Pad, Mounting_Holes:MountingHole_2.7mm_M2.5_ISO14580_Pad, F.Cu at (452.1, 110.1)
- added REF**: MountingHole_2.7mm_M2.5_ISO14580_Pad, Mounting_Holes:MountingHole_2.7mm_M2.5_ISO14580_Pad, F.Cu at (346.6, 45.2)
- added REF**: MountingHole_2.7mm_M2.5_ISO14580_Pad, Mounting_Holes:MountingHole_2.7mm_M2.5_ISO14580_Pad, F.Cu at (255.1, 45.2)
- added U17: MCP9804_MSOP, Housings_SSOP:MSOP-8_3x3mm_Pitch0.65mm, F.Cu at (162.7, 297.2)
- added U17: MCP9804_MSOP, Housings_SSOP:MSOP-8_3x3mm_Pitch0.65mm, F.Cu at (300.6, 77.5)
- added U18: MCP9804_MSOP, Housings_SSOP:MSOP-8_3x3mm_Pitch0.65mm, F.Cu at (496.4, 75.1)
- added U18: MCP9804_MSOP, Housings_SSOP:MSOP-8_3x3mm_Pitch0.65mm, F.Cu at (162.7, 179.6)
- added U19: ADC084S051, Housings_SSOP:MSOP-10_3x3mm_Pitch0.5mm, F.Cu at (77.2, 113.2)
- moved C1 74.4 mm to (60.4, 50.8)
- moved C11 74.4 mm to (92.8, 118.7)
- moved C19 74.4 mm to (92.8, 109.8)
- moved C24 74.4 mm to (106.1, 63.2)
- moved J5 74.4 mm to (61.9, 127.5)
- moved JP9 74.4 mm to (87.8, 123.4)
- moved U12 74.4 mm to (55.4, 84.2)
- moved U7 74.4 mm to (93.3, 123.6)
- moved C12 74.4 mm to (94.0, 118.7)
- moved C13 74.4 mm to (99.5, 118.7)
- moved C15 74.4 mm to (52.0, 118.7)
- moved C36 74.4 mm to (106.1, 112.1)
- moved C39 74.4 mm to (48.8, 95.2)
- moved C5 74.4 mm to (49.5, 61.9)
- moved C7 74.4 mm to (89.5, 114.0)
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Connections:
- J1 pad 11: Net-(J1-Pad11) -> FOD_DPL
- J1 pad 15: MAG_EN -> FOD_CC
- J1 pad 29: Net-(J1-Pad29) -> MAG_EN
- J6 pad 7: FOD_VAUX -> FOD_3V3
Routing:
- net MAG_3V3: track 115.0 -> 580.0 mm, vias 2 -> 10
- net RPI_SCL: track 120.3 -> 449.9 mm, vias 0 -> 4
- net RPI_SDA: track 121.8 -> 366.6 mm, vias 0 -> 8
- net FOD_CC: track 0.00 -> 74.7 mm, vias 0 -> 2
- net MAG2_BIT1: track 0.00 -> 72.0 mm
- net MAG2_BIT0: track 0.00 -> 64.4 mm
- net MAG1_BIT1: track 0.00 -> 64.2 mm
- net MAG1_BIT0: track 0.00 -> 57.5 mm
- net MAG1_A2: track 0.00 -> 57.5 mm
- net MAG2_A2: track 0.00 -> 53.7 mm
- net FOD_DPL: track 0.00 -> 52.4 mm, vias 0 -> 2
- net MAG1_A1: track 0.00 -> 40.5 mm
- net MAG2_A1: track 0.00 -> 40.1 mm
- net MAG2_A0: track 0.00 -> 30.6 mm
- net MAG1_A0: track 0.00 -> 29.5 mm
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Other:
- board size 92.5 x 86.8 mm -> 522.8 x 310.4 mm
- board text added: "SPEL - University of Chile - 2021"
- board text added: "Sensor Board PC104 V1 Serial"

Commit message: add langmuir probe
Parts:
- added J16: Conn_01x06_Male, Connectors_Molex:Molex_PicoBlade_53047-0610_06x1.25mm_Straight, F.Cu at (43.0, 262.3)
- added J16: Conn_01x06_Male, Connectors_Molex:Molex_PicoBlade_53047-0610_06x1.25mm_Straight, F.Cu at (43.1, 155.2)
- added J17: Conn_02x05_Counter_Clockwise, Pin_Headers:Pin_Header_Angled_2x05_Pitch1.27mm, B.Cu at (43.9, 173.0)
- added J18: Conn_01x06_Male, Pin_Headers:Pin_Header_Straight_1x06_Pitch2.54mm, B.Cu at (110.0, 280.1)
- added J18: Conn_01x06_Male, Pin_Headers:Pin_Header_Straight_1x06_Pitch2.54mm, B.Cu at (110.1, 172.9)
- added J19: Conn_01x03_Male, Pin_Headers:Pin_Header_Straight_1x03_Pitch2.54mm, B.Cu at (102.5, 260.0)
- added J19: Conn_01x03_Male, Pin_Headers:Pin_Header_Straight_1x03_Pitch2.54mm, B.Cu at (102.6, 152.7)
- added J20: Conn_01x03_Male, Pin_Headers:Pin_Header_Straight_1x03_Pitch2.54mm, B.Cu at (92.4, 260.0)
- added J20: Conn_01x03_Male, Pin_Headers:Pin_Header_Straight_1x03_Pitch2.54mm, B.Cu at (92.5, 152.7)
- added J21: Conn_01x06_Male, Pin_Headers:Pin_Header_Straight_1x06_Pitch2.54mm, B.Cu at (69.1, 297.5)
- added J21: Conn_01x06_Male, Pin_Headers:Pin_Header_Straight_1x06_Pitch2.54mm, B.Cu at (69.2, 190.3)
- added J22: Conn_01x03_Male, Pin_Headers:Pin_Header_Straight_1x03_Pitch2.54mm, B.Cu at (82.3, 260.0)
- added J22: Conn_01x03_Male, Pin_Headers:Pin_Header_Straight_1x03_Pitch2.54mm, B.Cu at (82.4, 152.7)
- added J23: Conn_01x03_Male, Pin_Headers:Pin_Header_Straight_1x03_Pitch2.54mm, B.Cu at (72.2, 260.0)
- added J23: Conn_01x03_Male, Pin_Headers:Pin_Header_Straight_1x03_Pitch2.54mm, B.Cu at (72.3, 152.7)
- added J24: Conn_01x06_Male, Pin_Headers:Pin_Header_Straight_1x06_Pitch2.54mm, B.Cu at (59.6, 267.4)
- added J24: Conn_01x06_Male, Pin_Headers:Pin_Header_Straight_1x06_Pitch2.54mm, B.Cu at (59.7, 160.2)
- added JP29: Jumper_3_Open, Jumper:SolderJumper-3_P1.3mm_Open_RoundedPad1.0x1.5mm, F.Cu at (99.9, 264.2)
- added JP29: Jumper_3_Open, Jumper:SolderJumper-3_P1.3mm_Open_RoundedPad1.0x1.5mm, F.Cu at (100.0, 157.0)
- added JP30: Jumper_3_Open, Jumper:SolderJumper-3_P1.3mm_Open_RoundedPad1.0x1.5mm, F.Cu at (89.8, 264.2)
- added JP30: Jumper_3_Open, Jumper:SolderJumper-3_P1.3mm_Open_RoundedPad1.0x1.5mm, F.Cu at (89.9, 157.0)
- added JP31: Jumper_3_Open, Jumper:SolderJumper-3_P1.3mm_Open_RoundedPad1.0x1.5mm, F.Cu at (79.9, 264.2)
- added JP31: Jumper_3_Open, Jumper:SolderJumper-3_P1.3mm_Open_RoundedPad1.0x1.5mm, F.Cu at (80.0, 157.0)
- added JP32: Jumper_3_Open, Jumper:SolderJumper-3_P1.3mm_Open_RoundedPad1.0x1.5mm, F.Cu at (69.6, 264.2)
- added JP32: Jumper_3_Open, Jumper:SolderJumper-3_P1.3mm_Open_RoundedPad1.0x1.5mm, F.Cu at (69.8, 157.0)
Routing:
- net LPS_5V: track 0.00 -> 334.1 mm
- net GND: track 208.2 -> 246.2 mm
- net VPOS: track 0.00 -> 10.2 mm
- net VNEG: track 0.00 -> 10.2 mm
- net ENP: track 0.00 -> 8.58 mm
- net PSP: track 0.00 -> 8.56 mm
- net PSN: track 0.00 -> 8.51 mm
- net ENN: track 0.00 -> 8.46 mm
Other:
- board text added: "3V3"
- board text added: "5V"
- board text added: "AOA SPI"
- board text added: "CC"
- board text added: "CLK"
- board text added: "CS"
- board text added: "DPL"
- board text added: "FOD SPI"
- board text added: "GND"
- board text added: "Isolated"
- board text added: "MISO"
- board text added: "MOSI"
- board text added: "OUT1"
- board text added: "OUT2"
- board text added: "OUT3"
- board text added: "OUT4"
- board text added: "OUT5"
- board text added: "OUT6"
- board text added: "PIC EN"
- board text added: "SCK"
- board text added: "SCL"
- board text added: "SDA"
- board text added: "Sensor Board Panel A S2 E V1 Serial"
- board text added: "Sensor Board Panel A S2 I V1 Serial"
- board text added: "Sensor Board Panel A S3 E V1 Serial"
- board text added: "Sensor Board Panel A S3 I V1 Serial"
- board text added: "Sensor Board Panel B E S3 V1 Serial"
- board text added: "Sensor Board Panel B I S3 V1 Serial"
- board text added: "Sensor Board Panel B S2 E V1 Serial"
- board text added: "Sensor Board Panel B S2 I V1 Serial"

Commit message: PCB update
Parts:
- removed J10 (x2), J11 (x2): Conn_01x04_Male, Connectors_Molex:Molex_PicoBlade_53398-0471_04x1.25mm_Straight
- removed J12 (x2), J14 (x2): Conn_01x07_Female, Pin_Headers:Pin_Header_Straight_1x07_Pitch2.54mm_SMD_Pin1Left
- removed J13 (x2), J15 (x2): Conn_01x07_Female, Pin_Headers:Pin_Header_Straight_1x07_Pitch2.54mm_SMD_Pin1Right
- removed J16 (x2): Conn_01x06_Male, Connectors_Molex:Molex_PicoBlade_53047-0610_06x1.25mm_Straight
- removed J17: Conn_02x05_Counter_Clockwise, Pin_Headers:Pin_Header_Angled_2x05_Pitch1.27mm
- removed J18 (x2), J21 (x2), J24 (x2): Conn_01x06_Male, Pin_Headers:Pin_Header_Straight_1x06_Pitch2.54mm
- removed J19 (x2), J20 (x2), J22 (x2), J23 (x2): Conn_01x03_Male, Pin_Headers:Pin_Header_Straight_1x03_Pitch2.54mm
- removed JP19 (x2), JP20 (x2), JP21 (x2), JP22 (x2), JP23 (x2), JP24 (x2), JP25 (x2), JP26 (x2), JP27 (x2), JP28 (x2), JP29 (x2), JP30 (x2), JP31 (x2), JP32 (x2): Jumper_3_Open, Jumper:SolderJumper-3_P1.3mm_Open_RoundedPad1.0x1.5mm
- removed R16 (x2), R17 (x2), R18 (x2), R19 (x2): R, Resistors_SMD:R_0402
- removed the REF** at (553.3, 45.9)
- removed the REF** at (346.6, 109.4)
- removed the REF** at (242.8, 109.4)
- removed the REF** at (242.8, 45.2)
- removed the REF** at (151.3, 45.2)
- removed the REF** at (150.9, 109.4)
- removed the REF** at (336.1, 46.0)
- removed the REF** at (293.5, 108.6)
- removed the REF** at (293.5, 46.0)
- removed the REF** at (336.1, 108.6)
- removed the REF** at (194.2, 332.7)
- removed the REF** at (461.8, 45.9)
- removed the REF** at (131.6, 332.7)
- removed the REF** at (194.2, 290.1)
- removed the REF** at (131.6, 290.1)
- removed the REF** at (547.0, 53.4)
- removed the REF** at (547.0, 101.3)
- removed the REF** at (512.0, 42.8)
- removed the REF** at (512.0, 113.1)
- removed the REF** at (314.8, 107.8)
- removed the REF** at (314.8, 46.8)
- removed the REF** at (132.4, 311.4)
- removed the REF** at (553.3, 110.1)
- removed the REF** at (193.4, 311.4)
- removed the REF** at (201.0, 251.7)
- removed the REF** at (201.0, 343.3)
- removed the REF** at (124.8, 251.7)
- removed the REF** at (124.8, 343.3)
- removed the REF** at (115.3, 251.4)
- removed the REF** at (115.3, 343.0)
- removed the REF** at (39.1, 251.4)
- removed the REF** at (39.1, 343.0)
- removed the REF** at (115.4, 144.2)
- removed the REF** at (452.1, 45.9)
- removed the REF** at (115.4, 235.8)
- removed the REF** at (39.2, 144.2)
- removed the REF** at (39.2, 235.8)
- removed the REF** at (187.4, 230.1)
- removed the REF** at (139.6, 230.1)
- removed the REF** at (198.1, 195.1)
- removed the REF** at (127.8, 195.1)
- removed the REF** at (201.0, 235.8)
- removed the REF** at (124.8, 235.8)
- removed the REF** at (201.0, 144.2)
- removed the REF** at (360.6, 45.9)
- removed the REF** at (124.8, 144.2)
- removed the REF** at (360.6, 110.1)
- removed the REF** at (452.1, 110.1)
- removed the REF** at (346.6, 45.2)
- removed the REF** at (255.1, 45.2)
- removed U17 (x2), U18 (x2): MCP9804_MSOP, Housings_SSOP:MSOP-8_3x3mm_Pitch0.65mm
- moved C26 0.21 mm to (75.0, 116.1)
Routing:
- net MAG_3V3: track 580.0 -> 90.3 mm, vias 10 -> 2
- net LPS_5V: track 334.1 -> 0.00 mm
- net RPI_SCL: track 449.9 -> 121.5 mm, vias 4 -> 0
- net RPI_SDA: track 366.6 -> 122.3 mm, vias 8 -> 0
- net MAG2_BIT1: track 72.0 -> 0.00 mm
- net MAG2_BIT0: track 64.4 -> 0.00 mm
- net MAG1_BIT1: track 64.2 -> 0.00 mm
- net MAG1_BIT0: track 57.5 -> 0.00 mm
- net MAG1_A2: track 57.5 -> 0.00 mm
- net MAG2_A2: track 53.7 -> 0.00 mm
- net MAG1_A1: track 40.5 -> 0.00 mm
- net MAG2_A1: track 40.1 -> 0.00 mm
- net GND: track 246.2 -> 208.1 mm
- net MAG2_A0: track 30.6 -> 0.00 mm
- net MAG1_A0: track 29.5 -> 0.00 mm
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Other:
- board size 522.8 x 310.4 mm -> 92.5 x 86.8 mm
- board text removed: "Sensor Board Panel A S2 E V1 Serial"
- board text removed: "Sensor Board Panel A S2 I V1 Serial"
- board text removed: "Sensor Board Panel A S3 E V1 Serial"
- board text removed: "Sensor Board Panel A S3 I V1 Serial"
- board text removed: "Sensor Board Panel B E S3 V1 Serial"
- board text removed: "Sensor Board Panel B I S3 V1 Serial"
- board text removed: "Sensor Board Panel B S2 E V1 Serial"
- board text removed: "Sensor Board Panel B S2 I V1 Serial"

Commit message: Update PCBs
New version of PCBs
Parts:
- added JP33: Jumper_2_Open, Jumper:SolderJumper-2_P1.3mm_Open_RoundedPad1.0x1.5mm, F.Cu at (95.1, 51.5)
- added R12: R, Resistors_SMD:R_0402, F.Cu at (83.0, 113.3)
- added R14: R, Resistors_SMD:R_0402, F.Cu at (83.0, 114.5)
- added R20: R, Resistors_SMD:R_0402, F.Cu at (69.7, 113.0)
- added R21: R, Resistors_SMD:R_0402, F.Cu at (69.7, 111.7)
- R10, R7, R8, R9: footprint Resistors_SMD:R_0402 -> Resistors_SMD:R_0603
- U10, U7, U8, U9: footprint AD7904:QPQ1906SR -> AD7904:QPQ1906SR2
- moved J4 0.63 mm to (53.1, 127.7)
- moved J2 0.59 mm to (93.9, 127.7)
- moved J3 0.58 mm to (101.7, 127.7)
- moved J5 0.56 mm to (61.3, 127.7)
- moved R10 0.33 mm to (61.0, 120.6)
- moved R8 0.31 mm to (101.3, 120.6)
- moved R9 0.28 mm to (52.8, 120.6)
- moved R7 0.23 mm to (93.5, 120.6)
- moved U8 0.20 mm to (52.6, 123.6)
- moved U9 0.10 mm to (60.7, 123.3)
Connections:
- J1 pad 7: Net-(J1-Pad7) -> FOD_STS
- U19 pad 4: VPHS2 -> VPHS2A
- U19 pad 5: VMAG2 -> VMAG2A
- U19 pad 6: VPHS1 -> VPHS1A
- U19 pad 7: VMAG1 -> VMAG1A
Routing:
- net GND: track 208.1 -> 252.4 mm, vias 15 -> 46
- net FOD_STS: track 0.00 -> 31.5 mm, vias 0 -> 1
- net VPHS2: track 25.3 -> 18.8 mm
- net VMAG2: track 28.0 -> 21.5 mm
- net FOD_SDA: track 4.34 -> 10.5 mm
- net VPHS2A: track 0.00 -> 5.65 mm
- net VMAG2A: track 0.00 -> 5.30 mm
- net VMAG1: track 23.8 -> 19.5 mm
- net VPHS1: track 25.5 -> 21.8 mm
- net VMAG1A: track 0.00 -> 3.33 mm
- net VPHS1A: track 0.00 -> 3.32 mm
- net FOD_3V3: track 98.1 -> 99.2 mm
- net ANT3_IN: track 2.84 -> 2.33 mm
- net (no net): vias 0 -> 1
Other:
- board text added: "ISC CLK"
- board text added: "ISC DAT"
- board text added: "MCLR"
- board text added: "PIC 3V3"
- board text added: "STS"
- board text added: "Sensor Board PC104 V1.11 Serial"
- board text removed: "Sensor Board PC104 V1 Serial"

Commit message: minor changes
Connections:
- U1 pad 81: Net-(U1-Pad81) -> GND
- U1 pad 82: Net-(U1-Pad82) -> GND
- U1 pad 84: Net-(U1-Pad84) -> GND
Routing:
- net GND: track 252.4 -> 382.8 mm, vias 46 -> 44
- net (no net): track 0.00 -> 2.47 mm
