File: A/Hardware/Panel A E S2/MAG_Plus/MAG_Plus.kicad_pcb (KiCad board)
At the start: 2 copper layers, 82.6 x 98 mm, 20 parts, among them J11 Conn_01x04_Male, J13 Conn_01x07_Female, J15 Conn_01x07_Female, U18 MCP9804_MSOP

Commit message: Update PCBs
New version of PCBs
Parts:
- removed the REF** at (187.4, 230.1)
- removed the REF** at (138.9, 230.1)
- removed the REF** at (198.1, 196.0)
- added G***: LOGO, L86:FCFM, B.Cu at (163.9, 212.1)
- added REF**: MountingHole_2.2mm_M2_DIN965, Mounting_Holes:MountingHole_2.2mm_M2_DIN965, F.Cu at (195.9, 222.9)
- added REF**: MountingHole_2.2mm_M2_DIN965, Mounting_Holes:MountingHole_2.2mm_M2_DIN965, F.Cu at (129.8, 222.9)
- added REF**: MountingHole_2.2mm_M2_DIN965, Mounting_Holes:MountingHole_2.2mm_M2_DIN965, F.Cu at (195.9, 203.1)
- added REF**: MountingHole_2.2mm_M2_DIN965, Mounting_Holes:MountingHole_2.2mm_M2_DIN965, F.Cu at (129.8, 203.1)
- added REF**: MountingHole_2.7mm_M2.5_ISO14580_Pad, Mounting_Holes:MountingHole_2.7mm_M2.5_ISO14580_Pad, F.Cu at (187.2, 230.0)
- added REF**: MountingHole_2.7mm_M2.5_ISO14580_Pad, Mounting_Holes:MountingHole_2.7mm_M2.5_ISO14580_Pad, F.Cu at (138.7, 230.0)
- added REF**: MountingHole_2.7mm_M2.5_ISO14580_Pad, Mounting_Holes:MountingHole_2.7mm_M2.5_ISO14580_Pad, F.Cu at (198.1, 196.0)
- moved G*** 43.3 mm to (163.0, 169.2), turned to 180 degrees
Other:
- board text added: "1 - 0"
- board text added: "MAG 1|0"
- board text added: "Sensor Board Panel A S2 E V1.1 Serial"
- board text added: "TEMP 2|1|0"
- board text removed: "Sensor Board Panel A S2 E V1 Serial"
