File: A/Hardware/Panel A I S2/MAG_Plus/MAG_Plus.kicad_pcb (KiCad board)
At the start: 2 copper layers, 82.6 x 98 mm, 18 parts, among them J16 Conn_01x06_Male, J17 Conn_02x05_Counter_Clockwise, J18 Conn_01x06_Male, J19 Conn_01x03_Male, J20 Conn_01x03_Male, J21 Conn_01x06_Male, J22 Conn_01x03_Male, J23 Conn_01x03_Male, J24 Conn_01x06_Male

Commit message: Update PCBs
New version of PCBs
Parts:
- JP33: moved to F.Cu
- moved JP33 10.7 mm to (57.0, 153.6)
- moved J16 4.87 mm to (43.1, 150.3)
- moved J17 3.06 mm to (45.8, 170.5)
Routing:
- net GND: track 40.2 -> 72.0 mm
- net VNEG: track 70.4 -> 95.3 mm, vias 1 -> 0
- net LPS_TX: track 22.2 -> 43.9 mm
- net LPS_RX: track 20.2 -> 33.9 mm
- net LPS_3V3: track 3.77 -> 12.8 mm
- net VPOS: track 52.7 -> 44.5 mm, vias 1 -> 0
- net LPS_3V3J: track 20.6 -> 28.6 mm, vias 0 -> 1
- net LPS_5V: track 183.2 -> 188.3 mm
Other:
- board text added: "Sensor Board Panel A S2 I V1.1 Serial"
- board text removed: "Sensor Board Panel A S2 I V1 Serial"
