File: A/Hardware/Panel B E S2/MAG_Plus/MAG_Plus.kicad_pcb (KiCad board)
At the start: 2 copper layers, 98 x 82.6 mm, 19 parts, among them J11 Conn_01x04_Male, J13 Conn_01x07_Female, J15 Conn_01x07_Female, U18 MCP9804_MSOP

Commit message: Update PCBs
New version of PCBs
Parts:
- added REF**: MountingHole_2.7mm_M2.5_ISO14580_Pad, Mounting_Holes:MountingHole_2.7mm_M2.5_ISO14580_Pad, F.Cu at (468.5, 86.3)
Changed lines of the file:
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@@
     (tracks 172)
     (zones 0)
-    (modules 19)
+    (modules 20)
     (nets 16)
   )
@@
     (add_net RPI_SDA)
   )
+  (module Mounting_Holes:MountingHole_2.7mm_M2.5_ISO14580_Pad (layer F.Cu)
+    (at 468.49 86.27)
+    (descr "Mounting Hole 2.7mm, M2.5, ISO14580")
+    (tags "mounting hole 2.7mm m2.5 iso14580")
+    (attr virtual)
+    (fp_text reference REF** (at 0 -3.25) (layer F.SilkS)
+      (effects (font (size 1 1) (thickness 0.15)))
+    )
+    (fp_text value MountingHole_2.7mm_M2.5_ISO14580_Pad (at 0 3.25) (layer F.Fab)
+      (effects (font (size 1 1) (thickness 0.15)))
+    )
+    (fp_circle (center 0 0) (end 2.5 0) (layer F.CrtYd) (width 0.05))
+    (fp_circle (center 0 0) (end 2.25 0) (layer Cmts.User) (width 0.15))
+    (fp_text user %R (at 0.3 0) (layer F.Fab)
+      (effects (font (size 1 1) (thickness 0.15)))
+    )
+    (pad 1 thru_hole circle (at 0 0) (size 4.5 4.5) (drill 2.7) (layers *.Cu *.Mask))
+  )
   (module L86:SPEL_logo (layer B.Cu)
