File: A/Hardware/Panel B I S3/MAG_Plus/MAG_Plus.kicad_pcb (KiCad board)
At the start: 2 copper layers, 98 x 82.6 mm, 4 parts

Commit message: Update PCBs
New version of PCBs
Parts:
- added REF**: pad, L86:pad, B.Cu at (168.5, 64.2)
- added REF**: pad, L86:pad, F.Cu at (168.6, 64.2)
Routing:
- net (no net): vias 0 -> 1
Other:
- outline, holes or cut-outs redrawn
- board text added: "Sensor Board Panel B I S3 V1.1 Serial"
- board text removed: "Sensor Board Panel B I S3 V1 Serial"
Changed lines of the file:
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@@
   (general
     (thickness 1.6)
-    (drawings 43)
-    (tracks 0)
+    (drawings 52)
+    (tracks 1)
     (zones 0)
-    (modules 4)
+    (modules 6)
     (nets 2)
   )
@@
     (uvia_drill 0.1)
   )
+  (module L86:pad (layer B.Cu)
+    (at 168.48 64.17 270)
+    (fp_text reference REF** (at 0 -0.5 270) (layer B.SilkS)
+      (effects (font (size 1 1) (thickness 0.15)) (justify mirror))
+    )
+    (fp_text value pad (at 0 0.5 270) (layer B.Fab)
+      (effects (font (size 1 1) (thickness 0.15)) (justify mirror))
+    )
+    (pad 1 smd rect (at 0 -0.1 270) (size 26.3 3) (layers B.Cu B.Paste B.Mask))
+  )
+  (module L86:pad (layer F.Cu)
+    (at 168.55 64.16 90)
+    (fp_text reference REF** (at 0 0.5 90) (layer F.SilkS)
+      (effects (font (size 1 1) (thickness 0.15)))
+    )
+    (fp_text value pad (at 0 -0.5 90) (layer F.Fab)
+      (effects (font (size 1 1) (thickness 0.15)))
+    )
+    (pad 1 smd rect (at 0 0.03 90) (size 26.3 3) (layers F.Cu F.Paste F.Mask))
+  )
   (module Mounting_Holes:MountingHole_2.7mm_M2.5_ISO14580_Pad (layer F.Cu)
     (at 242.8 107.81)
@@
     (pad 1 thru_hole circle (at 0 0) (size 4.5 4.5) (drill 2.7) (layers *.Cu *.Mask))
   )
+  (gr_line (start 210.35 39.2) (end 234 39.2) (layer Edge.Cuts) (width 0.05))
+  (gr_line (start 210.35 115.4) (end 234 115.4) (layer Edge.Cuts) (width 0.05))
+  (gr_line (start 210.35 103.6) (end 210.35 39.2) (layer Edge.Cuts) (width 0.05))
+  (gr_line (start 210.35 103.6) (end 210.35 115.4) (layer Edge.Cuts) (width 0.05))
+  (gr_line (start 170.35 103.6) (end 210.35 103.6) (layer F.SilkS) (width 0.12))
+  (gr_line (start 166.99 77.51) (end 167 51) (layer Edge.Cuts) (width 0.05))
+  (gr_line (start 170.36 103.6) (end 170.36 96.81) (layer Edge.Cuts) (width 0.05))
+  (gr_line (start 167 103.6) (end 170.36 103.6) (layer Edge.Cuts) (width 0.05))
+  (gr_line (start 170.36 88.93) (end 170.36 96.81) (layer Edge.Cuts) (width 0.05))
+  (gr_line (start 170.37 77.52) (end 170.36 88.93) (layer Edge.Cuts) (width 0.05))
+  (gr_line (start 166.99 77.51) (end 170.37 77.52) (layer Edge.Cuts) (width 0.05))
+  (gr_line (start 153 51) (end 153 103.6) (layer Edge.Cuts) (width 0.05))
+  (gr_line (start 167 51) (end 153 51) (layer Edge.Cuts) (width 0.05))
+  (gr_line (start 153 103.6) (end 167 103.6) (layer Edge.Cuts) (width 0.05))
+  (gr_line (start 167 103.6) (end 153 103.6) (layer F.SilkS) (width 0.12))
+  (gr_line (start 153 51) (end 167.01 51) (layer F.SilkS) (width 0.12))
+  (gr_line (start 167.01 51) (end 153 51) (layer F.SilkS) (width 0.12))
+  (dimension 15 (width 0.12) (layer F.SilkS)
+    (gr_text "15.000 mm" (at 151.73 43.5 270) (layer F.SilkS)
+      (effects (font (size 1 1) (thickness 0.15)))
+    )
+    (feature1 (pts (xy 153 51) (xy 152.413579 51)))
+    (feature2 (pts (xy 153 36) (xy 152.413579 36)))
+    (crossbar (pts (xy 153 36) (xy 153 51)))
+    (arrow1a (pts (xy 153 51) (xy 152.413579 49.873496)))
+    (arrow1b (pts (xy 153 51) (xy 153.586421 49.873496)))
+    (arrow2a (pts (xy 153 36) (xy 152.413579 37.126504)))
+    (arrow2b (pts (xy 153 36) (xy 153.586421 37.126504)))
+  )
+  (gr_line (start 153 118.6) (end 153 36) (layer F.SilkS) (width 0.12))
   (gr_poly (pts (xy 205.72 41.91) (xy 205.72 46.91) (xy 200.72 46.91) (xy 200.72 41.91)) (layer F.SilkS) (width 0.1))
   (gr_poly (pts (xy 199.72 41.91) (xy 199.72 46.91) (xy 194.72 46.91) (xy 194.72 41.91)) (layer F.SilkS) (width 0.1))
@@
     (effects (font (size 1 1) (thickness 0.15)))
   )
-  (gr_text "Sensor Board Panel B I S3 V1 Serial" (at 194.17 48.31) (layer F.SilkS)
+  (gr_text "Sensor Board Panel B I S3 V1.1 Serial" (at 194.17 48.31) (layer F.SilkS)
     (effects (font (size 1 1) (thickness 0.15)))
   )
-  (gr_line (start 234 115.4) (end 208 115.4) (layer Edge.Cuts) (width 0.05))
   (gr_line (start 234.01 104.8) (end 234 115.4) (layer Edge.Cuts) (width 0.05))
   (gr_line (start 239.6 104.8) (end 234.01 104.8) (layer Edge.Cuts) (width 0.05))
@@
   (gr_line (start 234 49.8) (end 239.6 49.8) (layer Edge.Cuts) (width 0.05))
   (gr_line (start 234 39.2) (end 234 49.8) (layer Edge.Cuts) (width 0.05))
-  (gr_line (start 208 39.2) (end 234 39.2) (layer Edge.Cuts) (width 0.05))
-  (gr_line (start 208 115.4) (end 208 39.2) (layer Edge.Cuts) (width 0.05))
   (gr_line (start 160 118.6) (end 160 104.8) (layer F.SilkS) (width 0.12))
   (gr_line (start 154.4 115.4) (end 239.6 115.4) (layer F.SilkS) (width 0.12))
-  (gr_line (start 183.22 115.4) (end 183.24 89.2) (layer Edge.Cuts) (width 0.05))
-  (gr_line (start 160 115.4) (end 183.22 115.4) (layer Edge.Cuts) (width 0.05))
-  (gr_line (start 160 104.8) (end 160 115.4) (layer Edge.Cuts) (width 0.05))
-  (gr_line (start 154.42 104.8) (end 160 104.8) (layer Edge.Cuts) (width 0.05))
-  (gr_line (start 154.44 89.2) (end 154.42 104.8) (layer Edge.Cuts) (width 0.05))
-  (gr_line (start 183.24 89.2) (end 154.44 89.2) (layer Edge.Cuts) (width 0.05))
   (gr_line (start 234 104.8) (end 234 118.6) (layer F.SilkS) (width 0.12))
   (gr_line (start 246 104.8) (end 234 104.8) (layer F.SilkS) (width 0.12))
@@
   (gr_line (start 239.6 39.2) (end 154.5 39.2) (layer F.SilkS) (width 0.12))
   (gr_line (start 239.6 36) (end 239.6 118.6) (layer F.SilkS) (width 0.12))
-  (gr_line (start 154.5 36) (end 154.4 118.6) (layer F.SilkS) (width 0.12))
   (gr_circle (center 242.8 107.8) (end 244.05 107.8) (layer F.SilkS) (width 0.12))
   (gr_circle (center 242.8 46.8) (end 244.05 46.8) (layer F.SilkS) (width 0.12))
@@
   (gr_line (start 148 118.6) (end 246 118.6) (layer Edge.Cuts) (width 0.05))
   (gr_line (start 148.1 36) (end 148 118.6) (layer Edge.Cuts) (width 0.05))
+  (via (at 267.94 67.69) (size 0.8) (drill 0.4) (layers F.Cu B.Cu) (net 0))
   (zone (net 1) (net_name GND) (layer F.Cu) (hatch edge 0.508)
     (connect_pads (clearance 0.508))
