File: A/Hardware/Panel B I S3/MAG_Plus/MAG_Plus.sch (KiCad schematic (older format))
At the start: 39 parts, among them J1 RPi_GPIO, J9 Conn_01x06_Male, SW1 SW_Push, U1 Payload, U12 PIC16F1847-I_SO, U13 LP38693MP-3.3, U14 LP38693MP-3.3, U15 LP38693MP-5.0, U16 LP38693MP-3.3, U2 ISO1540

Commit message: minor changes
Changed lines of the file:
@@
 $Descr A4 11693 8268
 encoding utf-8
-Sheet 1 5
+Sheet 1 6
 Title ""
 Date ""
@@
 F1 "LPS.sch" 50
 $EndSheet
+$Sheet
+S 10650 5950 500  150
+U 61B06CFF
+F0 "PC" 50
+F1 "PC.sch" 50
+$EndSheet
 $EndSCHEMATC
