File: A/Hardware/Panel B E S3/MAG_Plus/MAG_Plus.kicad_pcb (KiCad board)
At the start: 2 copper layers, 98 x 82.6 mm, 20 parts, among them J10 Conn_01x04_Male, J12 Conn_01x07_Female, J14 Conn_01x07_Female, U17 MCP9804_MSOP

Commit message: Update PCBs
New version of PCBs
Parts:
- removed the REF** at (314.8, 107.8)
- removed the REF** at (314.8, 46.8)
- added REF**: MountingHole_5.3mm_M5_DIN965_Pad, Mounting_Holes:MountingHole_5.3mm_M5_DIN965_Pad, F.Cu at (283.9, 108.4)
- added REF**: MountingHole_2.7mm_M2.5_ISO14580_Pad, Mounting_Holes:MountingHole_2.7mm_M2.5_ISO14580_Pad, F.Cu at (255.1, 107.8)
- moved J10 19.2 mm to (287.8, 53.5), turned to 0 degrees
Routing:
- net MAG_3V3: track 137.4 -> 121.1 mm
- net RPI_SCL: track 70.7 -> 55.4 mm
- net RPI_SDA: track 57.7 -> 45.4 mm
- net GND: track 41.6 -> 40.3 mm
Other:
- outline, holes or cut-outs redrawn
- board text added: "Sensor Board Panel B E S3 V1.1 Serial"
- board text removed: "Sensor Board Panel B E S3 V1 Serial"

Commit message: minor changes
Parts:
- J10, J12, J14, JP19, JP21, JP25, JP26, JP28, R17, R19, REF** (x9), U17: moved to B.Cu
- moved REF** 255.0 mm to (96.3, 22.0), turned to 270 degrees
- moved REF** 255.0 mm to (53.7, 22.0), turned to 270 degrees
- moved REF** 254.5 mm to (106.8, 22.8)
- moved REF** 254.5 mm to (15.3, 22.8)
- moved REF** 252.7 mm to (46.1, 23.0)
- moved JP26 249.3 mm to (59.5, 31.2)
- moved JP21 247.8 mm to (67.0, 34.1)
- moved JP28 247.8 mm to (59.4, 34.1)
- moved JP19 246.4 mm to (67.0, 37.0)
- moved JP25 246.4 mm to (59.4, 37.0)
- moved J14 244.4 mm to (60.7, 41.8), turned to 270 degrees
- moved REF** 242.9 mm to (96.3, 84.6), turned to 270 degrees
- moved REF** 242.9 mm to (53.7, 84.6), turned to 270 degrees
- moved REF** 242.7 mm to (15.3, 83.8)
- moved REF** 242.7 mm to (106.8, 83.8)
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Routing:
- added copper zone on F.Cu, net (none)
- added copper zone on B.Cu, net GND
- removed copper zone on B.Cu, net (none)
- removed copper zone on F.Cu, net GND
Other:
- outline, holes or cut-outs redrawn
